File: CAD/Eagle/DL0WH_BiTuner_MCU_1V0.sch (EAGLE design)
At the start: 133 parts, among them Q0321 ABS07-32.768KHZ, U0101 STM32L476RXT_64PIN_LDO, U2401 LM53603-Q1, U8921 TS5A23166, U8951 OPA354, U9001 TPS62051, U9401 MC33996, U9501 MC33996, U9601 MC33996, U9801 MAX232_SOIC16, U9901 MAX232_SOIC16, X2411 WIRE-TO-BOARD_5MM08_1X02, X3201 MOLEX 105017-0001, X3301 SMA_SMT_AMPHENOL-901-143, X3311 SAMTEC SMA-J-P-H-RA-TH1, X9851 WIRE-TO-BOARD_5MM08_1X02, X9852 WIRE-TO-BOARD_5MM08_1X02, X9853 WIRE-TO-BOARD_5MM08_1X02, X9951 WIRE-TO-BOARD_5MM08_1X02, X9952 WIRE-TO-BOARD_5MM08_1X02, X9953 WIRE-TO-BOARD_5MM08_1X02

Commit message: HW_1V0 - CAD/Eagle - pages renumbered: 17 pages
Parts:
- removed R9611: 47R, df4iah_rcl:R-EU_R0402
- added R0511: 1kR, df4iah_rcl:R-EU_R0402
- R0611: value 1kR -> 47R
- renumbered C2401 to C1201, C2402 to C1202, C2403 to C1203, C2404 to C1204, C2405 to C1205, C2411 to C1211, C2412 to C1212, C2421 to C1221, C2422 to C1222, C2423 to C1223, C3203 to C1403, C8901 to C0901, C8911 to C0911, C8921 to C0921, C8951 to C0951, C9001 to C1301, C9011 to C1311, C9401 to C0801, C9402 to C0802, C9403 to C0803, C9501 to C0701, C9502 to C0702, C9503 to C0703, C9601 to C0601, C9602 to C0602, C9603 to C0603, C9801 to C1001, C9802 to C1002, C9803 to C1003, C9804 to C1004, C9805 to C1005, C9901 to C1101, C9902 to C1102, C9903 to C1103, C9904 to C1104, C9905 to C1105, D8901 to D0901, D8911 to D0911, D8951 to D0951, D8961 to D0961, H3611 to H1711, H3621 to H1721, H3631 to H1731, H3651 to H1751, H3661 to H1761, L2411 to L1211, L8901 to L0901, L8911 to L0911, L9011 to L1311, PF3211 to PF1411, R0612 to R0512, R2411 to R1211, R3202 to R1402, R8901 to R0901, R8902 to R0902, R8903 to R0903, R8911 to R0911, R8912 to R0912, R8913 to R0913, R8921 to R0921, R8922 to R0922, R8951 to R0951, R8952 to R0952, R8961 to R0961, R9001 to R1301, R9002 to R1302, R9021 to R1321, R9022 to R1322, R9411 to R0811, R9424 to R0824, R9511 to R0711, R9524 to R0724, R9621 to R0621, R9622 to R0622, R9623 to R0623, R9624 to R0624, R9625 to R0625, R9626 to R0626, R9801 to R1001, R9802 to R1002, R9803 to R1003, R9804 to R1004, R9901 to R1101, R9902 to R1102, R9903 to R1103, R9904 to R1104, U2401 to U1201, U8921 to U0921, U8951 to U0951, U9001 to U1301, U9401 to U0801, U9501 to U0701, U9601 to U0601, U9801 to U1001, U9901 to U1101, X2411 to X1211, X3201 to X1401, X3301 to X1501, X3311 to X1511, X9701 to X1601, X9702 to X1602, X9851 to X1051, X9852 to X1052, X9853 to X1053, X9951 to X1151, X9952 to X1152, X9953 to X1153
Connections:
- net +3V3: now also R0511.2; no longer R0611.2
- net N$12: now also R0611.2; no longer R9611.2
- net PB9: now also R0511.1; no longer R0611.1
- net SPI_DRV_SO: now also R0611.1; no longer R9611.1

Commit message: HW_1V0 - 10uH Murata inductivity added
Signed-off-by: Ulrich Habel <espero7757@gmx.net>
Parts:
- L1311: device df4iah_rcl:L-EU4.90X4.90MM -> df4iah_rcl:L-EU4.50X3.20MM
Other:
- note added: "MURATA LQH43PN100M26L 4.5mm x 3.2mm (1812)"
- note removed: "MURATA LQH43PN100M26L 4.5mm x 3.2mm"
- note removed: "TODO !!!"
Changed lines of the file:
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@@
 <part name="R0824" library="df4iah_rcl" deviceset="R-EU_" device="R0402" value="47R"/>
 <part name="U1301" library="df4iah_powersupply" deviceset="TPS62051" device=""/>
-<part name="L1311" library="df4iah_rcl" deviceset="L-EU" device="4.90X4.90MM" value="10uH"/>
+<part name="L1311" library="df4iah_rcl" deviceset="L-EU" device="4.50X3.20MM" value="10uH"/>
 <part name="R1321" library="df4iah_rcl" deviceset="R-EU_" device="R0402" value="1MR"/>
 <part name="R1322" library="df4iah_rcl" deviceset="R-EU_" device="R0402" value="1MR"/>
@@
 <text x="157.48" y="96.52" size="1.778" layer="97">TPS_PG</text>
 <text x="157.48" y="91.44" size="1.778" layer="97">TPS_LBO</text>
-<text x="152.4" y="121.92" size="1.778" layer="97">MURATA  LQH43PN100M26L   4.5mm x 3.2mm</text>
-<text x="152.4" y="127" size="1.778" layer="97">TODO !!!</text>
+<text x="152.4" y="121.92" size="1.778" layer="97">MURATA  LQH43PN100M26L   4.5mm x 3.2mm (1812)</text>
 </plain>
 <instances>
