File: CAD/Eagle/DL0WH_BiTuner_Ctrl_1V0.brd (EAGLE design)
At the start: 96.5 x 73 mm, 141 parts, among them Q0321 ABS07-32.768KHZ, U0101 STM32L476RXT_64PIN_LDO, U0601 MC33996, U0701 MC33996, U0801 MC33996, U0921 TS5A23166, U0951 OPA354, U1001 MAX232_SOIC16, U1101 MAX232_SOIC16, U1201 LM53603-Q1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

Commit message: HW_1V0 HW_1V1 HW_1V2 - TPS62051 changed to TPS62056
Parts:
- U1301: value TPS62051 -> TPS62056
Changed lines of the file:
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@@
 <attribute name="VALUE" x="69.5325" y="12.7" size="0.6096" layer="27" font="vector" ratio="10" rot="R270"/>
 </element>
-<element name="U1301" library="df4iah_powersupply" package="S-PDSO-G10" value="TPS62051" x="15.24" y="39.37" rot="R180"/>
+<element name="U1301" library="df4iah_powersupply" package="S-PDSO-G10" value="TPS62056" x="15.24" y="39.37" rot="R180"/>
 <element name="L1311" library="df4iah_rcl" package="L_4.50MM_X_3.20MM" value="10uH" x="21.9075" y="36.83" smashed="yes" rot="R180">
 <attribute name="NAME" x="20.6375" y="38.735" size="0.6096" layer="25" font="vector" ratio="10"/>
