File: CAD/Eagle/DL0WH_BiTuner_Ctrl_1V3.sch (EAGLE design)
At the start: 157 parts, among them Q0321 ABS07-32.768KHZ, U0101 STM32L476RXT_64PIN_LDO, U0601 MC33996, U0701 MC33996, U0801 MC33996, U0921 TS5A23166, U0941 LM2611, U0951 OPA354, U0961 OPA354, U0962 MCP4661-103E-MS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

Commit message: HW_1V3 - forward until df4fd7a65716eb1a1b8dad1e9e020a2e6c04cd7f (2019-04-03)
Parts:
- removed C0054: 10nF, df4iah_rcl:C-EUC0603
- removed R0903, R0913: 150kR, df4iah_rcl:R-EU_R0402
- removed SJ0401: (no value), df4iah_jumper:SJ
- added C1054: 10nF, df4iah_rcl:C-EUC0402
- added R0401: 0R, df4iah_rcl:R-EU_R0402
- added R0923: 2MR, df4iah_rcl:R-EU_R0402
- C0942: device df4iah_rcl:C-EUC0805 -> df4iah_rcl:C-EUC0603
- C1051, C1052, C1053, C1151, C1152, C1153, C1154: device df4iah_rcl:C-EUC0603 -> df4iah_rcl:C-EUC0402
- R0962: value 1.0kR -> 1kR
- R0972: value 47R -> 1kR
- U0101: value STM32L476RXT_64PIN_LDO -> STM32L476RGT6_64PIN_LDO
- renumbered X0601 to X0501
Connections:
- net +3V3: now also R0401.1; no longer R0903.2, R0913.2, SJ0401.1
- net GND: now also C1054.2, R0923.1; no longer C0054.2
- net MCU_VDD: now also R0401.2; no longer SJ0401.2
- net RS_DTE_RTR: now also C1054.1; no longer C0054.1
- net SWR_IN_FWD: no longer R0903.1
- net SWR_IN_REV: no longer R0913.1
- net SWR_SEL_PWR: now also R0923.2
Other:
- note added: "nom: 4.9kR"
- note added: "nom: 5.0kR"
