File: CAD/Eagle/DL0WH_BiTuner_Ctrl_1V2.brd (EAGLE design)
At the start: 96.5 x 73 mm, 157 parts, among them Q0321 ABS07-32.768KHZ, U0101 STM32L476RXT_64PIN_LDO, U0601 MC33996, U0701 MC33996, U0801 MC33996, U0921 TS5A23166, U0941 LM2611, U0951 OPA354, U0961 OPA354, U0962 MCP4661-103E-MS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

Commit message: HW_1V2,HW_1V3 - CAD/Eagle - voltage divider added to tolerate voltages 0V..10V
Parts:
- C0901, C0911: value 1nF -> N/A
- L0901, L0911: value 10uH -> 2kR
- R0962: value 1.0kR -> 1kR
- R0963: value 10kR -> 20kR
Changed lines of the file:
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@@
 <layer number="27" name="tValues" color="7" fill="1" visible="no" active="yes"/>
 <layer number="28" name="bValues" color="7" fill="1" visible="no" active="yes"/>
-<layer number="29" name="tStop" color="7" fill="3" visible="yes" active="yes"/>
-<layer number="30" name="bStop" color="7" fill="6" visible="yes" active="yes"/>
-<layer number="31" name="tCream" color="7" fill="4" visible="yes" active="yes"/>
-<layer number="32" name="bCream" color="7" fill="5" visible="yes" active="yes"/>
+<layer number="29" name="tStop" color="7" fill="3" visible="no" active="yes"/>
+<layer number="30" name="bStop" color="7" fill="6" visible="no" active="yes"/>
+<layer number="31" name="tCream" color="7" fill="4" visible="no" active="yes"/>
+<layer number="32" name="bCream" color="7" fill="5" visible="no" active="yes"/>
 <layer number="33" name="tFinish" color="6" fill="3" visible="no" active="yes"/>
 <layer number="34" name="bFinish" color="6" fill="6" visible="no" active="yes"/>
@@
 <layer number="42" name="bRestrict" color="1" fill="10" visible="no" active="yes"/>
 <layer number="43" name="vRestrict" color="2" fill="10" visible="no" active="yes"/>
-<layer number="44" name="Drills" color="7" fill="1" visible="yes" active="yes"/>
+<layer number="44" name="Drills" color="7" fill="1" visible="no" active="yes"/>
 <layer number="45" name="Holes" color="7" fill="1" visible="no" active="yes"/>
 <layer number="46" name="Milling" color="3" fill="1" visible="yes" active="yes"/>
@@
 <layer number="49" name="Reference" color="7" fill="1" visible="yes" active="yes"/>
 <layer number="50" name="dxf" color="7" fill="1" visible="no" active="no"/>
-<layer number="51" name="tDocu" color="14" fill="1" visible="yes" active="yes"/>
-<layer number="52" name="bDocu" color="6" fill="1" visible="yes" active="yes"/>
+<layer number="51" name="tDocu" color="14" fill="1" visible="no" active="yes"/>
+<layer number="52" name="bDocu" color="6" fill="1" visible="no" active="yes"/>
 <layer number="53" name="tGND_GNDA" color="7" fill="9" visible="no" active="no"/>
 <layer number="54" name="bGND_GNDA" color="1" fill="9" visible="no" active="no"/>
@@
 <attribute name="VALUE" x="12.3825" y="36.5125" size="0.6096" layer="28" font="vector" ratio="10" rot="MR180"/>
 </element>
-<element name="L0901" library="df4iah_rcl" package="L0603" value="10uH" x="6.35" y="20.32" smashed="yes" rot="MR270">
+<element name="L0901" library="df4iah_rcl" package="L0603" value="2kR" x="6.35" y="20.32" smashed="yes" rot="MR270">
 <attribute name="NAME" x="10.16" y="18.0975" size="0.6096" layer="26" font="vector" ratio="10" rot="MR0"/>
 <attribute name="VALUE" x="7.9375" y="21.59" size="0.6096" layer="28" font="vector" ratio="10" rot="MR270"/>
 </element>
-<element name="L0911" library="df4iah_rcl" package="L0603" value="10uH" x="6.35" y="36.83" smashed="yes" rot="MR90">
+<element name="L0911" library="df4iah_rcl" package="L0603" value="2kR" x="6.35" y="36.83" smashed="yes" rot="MR90">
 <attribute name="NAME" x="10.16" y="38.4175" size="0.6096" layer="26" font="vector" ratio="10" rot="MR0"/>
 <attribute name="VALUE" x="4.7625" y="35.56" size="0.6096" layer="28" font="vector" ratio="10" rot="MR90"/>
 </element>
-<element name="C0901" library="df4iah_rcl" package="C0402" value="1nF" x="5.08" y="22.86" smashed="yes" rot="MR0">
+<element name="C0901" library="df4iah_rcl" package="C0402" value="N/A" x="5.08" y="22.86" smashed="yes" rot="MR0">
 <attribute name="NAME" x="3.175" y="22.5425" size="0.6096" layer="26" font="vector" ratio="10" rot="MR0"/>
 <attribute name="VALUE" x="6.35" y="21.2725" size="0.6096" layer="28" font="vector" ratio="10" rot="MR0"/>
 </element>
-<element name="C0911" library="df4iah_rcl" package="C0402" value="1nF" x="5.08" y="34.29" smashed="yes" rot="MR0">
+<element name="C0911" library="df4iah_rcl" package="C0402" value="N/A" x="5.08" y="34.29" smashed="yes" rot="MR0">
 <attribute name="NAME" x="3.175" y="33.9725" size="0.6096" layer="26" font="vector" ratio="10" rot="MR0"/>
 <attribute name="VALUE" x="6.35" y="32.7025" size="0.6096" layer="28" font="vector" ratio="10" rot="MR0"/>
@@
 <attribute name="VALUE" x="13.335" y="21.74875" size="0.6096" layer="28" font="vector" ratio="10" rot="MR270"/>
 </element>
-<element name="R0962" library="df4iah_rcl" package="R0402" value="1.0kR" x="11.7475" y="15.39875" rot="R270"/>
-<element name="R0963" library="df4iah_rcl" package="R0402" value="10kR" x="15.875" y="18.0975" smashed="yes" rot="MR90">
+<element name="R0962" library="df4iah_rcl" package="R0402" value="1kR" x="11.7475" y="15.39875" rot="R270"/>
+<element name="R0963" library="df4iah_rcl" package="R0402" value="20kR" x="15.875" y="18.0975" smashed="yes" rot="MR90">
 <attribute name="NAME" x="16.98625" y="16.8275" size="0.6096" layer="26" font="vector" ratio="10" rot="MR90"/>
 <attribute name="VALUE" x="14.2875" y="16.51" size="0.6096" layer="28" font="vector" ratio="10" rot="MR90"/>
